File: Malachi/281Project/Lab05.brd (EAGLE design)
At the start: 85.1 x 76.2 mm, 7 parts, among them X1 RASPI_BOARD_B+#_E4

Commit message: finished pcb
Parts:
- moved U$2 7.38 mm to (33.0, 20.1), turned to 0 degrees
Routing:
- net N$17: track 76.2 -> 106.5 mm
- net N$5: track 175.5 -> 156.4 mm
Changed lines of the file:
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@@
 <text x="21.59" y="46.99" size="1.778" layer="21" rot="R90">1K</text>
 <text x="31.75" y="49.53" size="1.778" layer="21" rot="R270">2K</text>
+<text x="0" y="35.306" size="1.778" layer="21">GPIO27</text>
+<text x="-0.254" y="32.512" size="1.778" layer="21">GPIO22</text>
+<text x="0.254" y="25.146" size="1.778" layer="21">GPIO5</text>
+<text x="0" y="22.606" size="1.778" layer="21">GPIO6</text>
 </plain>
 <attributes>
@@
 </element>
 <element name="U$1" library="mt280_21" package="DRV8835" value="DRV8835" x="56.388" y="37.592" smashed="yes" rot="R270"/>
-<element name="U$2" library="mt280_21" package="S13V20F5" value="S13V20F5" x="28.194" y="14.478" smashed="yes" rot="R90"/>
+<element name="U$2" library="mt280_21" package="S13V20F5" value="S13V20F5" x="33.02" y="20.066" smashed="yes"/>
 </elements>
 <signals>
@@
 <contactref element="U$2" pad="7"/>
 <wire x1="2.54" y1="52.07" x2="2.54" y2="12.7" width="1.016" layer="1"/>
-<wire x1="9.652" y1="5.588" x2="41.656" y2="5.588" width="1.016" layer="1"/>
-<wire x1="41.656" y1="5.588" x2="45.212" y2="9.144" width="1.016" layer="1"/>
-<wire x1="45.212" y1="9.144" x2="45.212" y2="17.018" width="1.016" layer="1"/>
-<wire x1="45.212" y1="17.018" x2="38.354" y2="17.018" width="1.016" layer="1"/>
-<wire x1="2.54" y1="12.7" x2="9.652" y2="5.588" width="1.016" layer="1"/>
+<wire x1="2.54" y1="12.7" x2="11.43" y2="3.81" width="1.016" layer="1"/>
+<wire x1="11.43" y1="3.81" x2="35.56" y2="3.81" width="1.016" layer="1"/>
+<wire x1="35.56" y1="3.81" x2="35.56" y2="9.906" width="1.016" layer="1"/>
 </signal>
 <signal name="N$6">
@@
 <contactref element="U$2" pad="9"/>
 <contactref element="X1" pad="2"/>
-<wire x1="38.354" y1="19.558" x2="38.354" y2="23.876" width="1.016" layer="16"/>
-<wire x1="38.354" y1="23.876" x2="21.336" y2="40.894" width="1.016" layer="16"/>
-<wire x1="21.336" y1="40.894" x2="21.336" y2="49.276" width="1.016" layer="16"/>
+<wire x1="48.055890625" y1="13.920109375" x2="47.895165625" y2="5.08" width="1.016" layer="16"/>
+<wire x1="47.895165625" y1="5.08" x2="42.926" y2="5.08" width="1.016" layer="16"/>
+<wire x1="38.1" y1="9.906" x2="42.926" y2="5.08" width="1.016" layer="16"/>
+<wire x1="48.055890625" y1="13.920109375" x2="21.336" y2="40.64" width="1.016" layer="16"/>
+<wire x1="21.336" y1="40.64" x2="21.336" y2="49.276" width="1.016" layer="16"/>
 <wire x1="21.336" y1="49.276" x2="12.319" y2="58.293" width="1.016" layer="16"/>
 <wire x1="12.319" y1="58.293" x2="12.192" y2="58.42" width="1.016" layer="16"/>
