File: Malachi/281Project/Lab05a.brd (EAGLE design)
At the start: 85.1 x 76.2 mm, 5 parts, among them X1 RASPI_BOARD_B+#_E4

Commit message: finished pcb
Parts:
- added SV2, SV4, SV5, SV8: (no value), con-lstb:MA03-1
- added SV6: (no value), con-lstb:MA05-1
- added SV7: (no value), con-lstb:MA07-1
- added U$1: DRV8835, mt280_21:DRV8835
- added U$2: S13V20F5, mt280_21:S13V20F5
- SV3: device con-lstb:MA06-1 -> con-lstb:MA03-1
- moved SV3 1.92 mm to (11.2, 31.8)
Connections:
- removed net 5V0A: X1.2
- removed net GND_C: X1.14
- removed net GND_H: X1.39
- new net 3V: SV2.3, SV3.3, SV4.3, SV5.3, U$1.2, X1.17
- new net GND: SV2.2, SV3.2, SV4.2, SV5.2, X1.25
- new net N$12: U$1.4, X1.33
- new net N$13: U$1.6, X1.32
- new net N$14: U$1.5, X1.37
- new net N$15: U$1.3, X1.35
- new net N$16: U$1.1, X1.39
- new net N$17: U$2.9, X1.2
- new net N$18: SV7.3, U$1.12
- new net N$19: SV7.4, U$1.11
- new net N$20: SV7.5, U$1.10
- new net N$21: SV7.6, U$1.9
- new net N$22: SV7.7, U$1.8
- new net N$23: SV6.5, U$2.1
- new net N$24: SV6.4, U$2.2
- new net N$25: SV6.3, U$2.3
- new net N$26: SV6.2, U$2.4
- new net N$27: SV6.1, U$2.5
- new net N$28: SV8.1, X1.12
- new net N$29: SV8.3, X1.14
- net N$1: now also SV8.2
- net N$10: now also SV5.1; no longer SV3.1
- net N$11: now also SV7.2, U$1.13; no longer SV3.3, X1.25
- net N$5: now also U$2.7
- net N$6: now also SV7.1, U$1.14; no longer SV3.4, X1.17
- net N$7: now also SV2.1; no longer SV3.6
- net N$8: now also SV3.1; no longer SV3.5
- net N$9: now also SV4.1; no longer SV3.2
Routing:
- net N$13: track 0.00 -> 140.6 mm
- net 3V: track 0.00 -> 132.9 mm
- net N$14: track 0.00 -> 116.7 mm
- net GND: track 0.00 -> 101.1 mm
- net N$17: track 0.00 -> 99.9 mm
- net N$5: track 74.3 -> 155.8 mm
- net N$27: track 0.00 -> 79.9 mm
- net N$11: track 66.1 -> 4.32 mm
- net N$25: track 0.00 -> 51.4 mm
- net N$6: track 50.4 -> 4.32 mm
- net N$24: track 0.00 -> 29.3 mm
- net N$23: track 0.00 -> 25.8 mm
- net N$26: track 0.00 -> 24.2 mm
- net N$1: track 31.7 -> 54.1 mm
- net N$15: track 0.00 -> 20.1 mm
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- added copper zone on layer 1, net GND
- added copper zone on layer 16, net GND
Other:
- board text added: "1K"
- board text added: "2K"
- board text added: "GPIO22"
- board text added: "GPIO27"
- board text added: "GPIO5"
- board text added: "GPIO6"
